File: szg-c2c-txr4.kicad_sch (KiCad schematic)
At the start: 37 parts, among them J1 SYZYGY_TXR-4, J2 SYZYGY_TXR-4, J3 Conn_01x02_Pin, U1 DSC557-0333

Commit message: change REFCLK circuit due to parts availability
Parts:
- removed U1: DSC557-0333, szg-c2c-txr4:VQFN14-2.5x3.2x0.9mm-EP1.4x2.1mm, symbol szg-c2c-txr4:DSC557-03
- added C22, C23: 8pF, Capacitor_SMD:C_0402_1005Metric, symbol Device:C_Small
- added J4: Conn_01x02_Pin, Connector_PinHeader_2.54mm:PinHeader_1x02_P2.54mm_Vertical, symbol Connector:Conn_01x02_Pin
- added R1, R4: 100Ω, Resistor_SMD:R_0402_1005Metric, symbol Device:R_Small_US
- added R2, R3, R5, R6: 150Ω, Resistor_SMD:R_0402_1005Metric, symbol Device:R_Small_US
- added R7: 470Ω, Resistor_SMD:R_0402_1005Metric, symbol Device:R_Small_US
- added U1: PI6C557-03, Package_SO:TSSOP-16_4.4x5mm_P0.65mm, symbol szg-c2c-txr4:PI6C557-03B
- added Y1: 25MHz 12pF, Crystal:Crystal_SMD_3225-4Pin_3.2x2.5mm, symbol Device:Crystal_GND24_Small
- C17: value 100nF -> 10nF
- FID1, FID2, FID3, FID4, FID5, FID6, FID7, FID8, H1, H2, H3, H4: now left out of the parts list
- J3: now not fitted
Connections:
- net +3V3: now also U1.12 (VDDA), U1.16 (VDDX), U1.6 (OE)
- net CLK0+: now also R1.1, R2.1, U1.15 (CLK0p)
- net CLK0-: now also R1.2, R3.1, U1.14 (CLK0n)
- net CLK1+: now also C20.1, R4.1, R5.1, U1.11 (CLK1p); no longer C21.1
- net CLK1-: now also C21.1, R4.2, R6.1, U1.10 (CLK1n); no longer C20.1
- net GND: now also C22.2, C23.2, J4.1 (Pin_1), R2.2, R3.2, R5.2, R6.2, R7.2, U1.13 (GNDA), U1.2 (S1), U1.7 (GNDX), Y1.2, Y1.4
- net J1_REFCLK+: now also C18.2; no longer C19.2
- net J1_REFCLK-: now also C19.2; no longer C18.2
- new net IREF: R7.1, U1.9 (IREF)
- new net SS1: J4.2 (Pin_2), U1.8 (SS1)
- new net X1: C22.1, U1.4 (X1/CLK), Y1.3
- new net X2: C23.1, U1.5 (X2), Y1.1
- no-connect marks 13 -> 16
Other:
- moved on the sheet: C17, C18, C19, C20, C21
